Commit message: fix:

File: lucia_description/urdf/turtlebot3_burger.urdf (robot description, URDF)
Before this commit: robot turtlebot3_burger, 7 links, 6 joints
Links:
- removed link ${namespace}base_footprint
- removed link ${namespace}base_link
- removed link ${namespace}base_scan
- removed link ${namespace}caster_back_link
- removed link ${namespace}imu_link
- removed link ${namespace}wheel_left_link
- removed link ${namespace}wheel_right_link
- added link base_footprint
- added link base_link, mass 8.2573504e-01; collision box size=0.140 0.140 0.143; visual mesh filename=package://turtlebot3_description/meshes/bases/burger_base.s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 scale=0.001 0.001 0.001
- added link base_scan, mass 0.114; collision cylinder length=0.0315 radius=0.055; visual mesh filename=package://turtlebot3_description/meshes/sensors/lds.stl scale=0.001 0.001 0.001
- added link caster_back_link, mass 0.005; collision box size=0.030 0.009 0.020
- added link imu_link
- added link wheel_left_link, mass 2.8498940e-02; collision cylinder length=0.018 radius=0.033; visual mesh filename=package://turtlebot3_description/meshes/wheels/left_tire.stl scale=0.001 0.001 0.001
- added link wheel_right_link, mass 2.8498940e-02; collision cylinder length=0.018 radius=0.033; visual mesh filename=package://turtlebot3_description/meshes/wheels/right_tire.s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 scale=0.001 0.001 0.001
Joints:
- removed joint ${namespace}base_joint
- removed joint ${namespace}caster_back_joint
- removed joint ${namespace}imu_joint
- removed joint ${namespace}scan_joint
- removed joint ${namespace}wheel_left_joint
- removed joint ${namespace}wheel_right_joint
- added joint base_joint: type fixed, parent base_footprint, child base_link, origin xyz=0.0 0.0 0.010 rpy=0 0 0
- added joint caster_back_joint: type fixed, parent base_link, child caster_back_link, origin xyz=-0.081 0 -0.004 rpy=-1.57 0 0
- added joint imu_joint: type fixed, parent base_link, child imu_link, origin xyz=-0.032 0 0.068 rpy=0 0 0
- added joint scan_joint: type fixed, parent base_link, child base_scan, origin xyz=-0.032 0 0.172 rpy=0 0 0
- added joint wheel_left_joint: type continuous, parent base_link, child wheel_left_link, origin xyz=0.0 0.08 0.023 rpy=-1.57 0 0, axis 0 0 1
- added joint wheel_right_joint: type continuous, parent base_link, child wheel_right_link, origin xyz=0.0 -0.080 0.023 rpy=-1.57 0 0, axis 0 0 1
