Commit message: fix: lucia_urdf

File: lucia_description/urdf/lucia.urdf (robot description, URDF)
Before this commit: robot lucia, 2 links, 1 joints
Links:
- added link base_footprint
- added link caster_wheel; visual sphere radius=0.05
- added link left_wheel; visual cylinder length=0.05 radius=0.1
- added link right_wheel; visual cylinder length=0.05 radius=0.1
- link base_link: geometry visual box size=0.6 0.4 0.2
- link base_scan: geometry visual cylinder length=0.06 radius=0.1
Joints:
- removed joint scan_joint
- added joint base_caster_wheel_joint: type fixed, parent base_link, child caster_wheel, origin xyz=0.2 0 -0.15 rpy=0 0 0
- added joint base_joint: type fixed, parent base_footprint, child base_link, origin xyz=0 0 0.2 rpy=0 0 0
- added joint base_left_wheel_joint: type continuous, parent base_link, child left_wheel, origin xyz=-0.1 0.2 -0.1 rpy=0 0 0, axis 0 1 0
- added joint base_right_wheel_joint: type continuous, parent base_link, child right_wheel, origin xyz=-0.1 -0.2 -0.1 rpy=0 0 0, axis 0 1 0
- added joint base_scan_joint: type fixed, parent base_link, child base_scan, origin xyz=0 0 0.13 rpy=0 0 0

Commit message: fix: lucia_urdf

File: lucia_description/urdf/lucia.urdf (robot description, URDF)
Before this commit: robot my_robot, 6 links, 5 joints
Links:
- link base_link: geometry visual cylinder length=1.0 radius=0.5
Joints:
- joint base_caster_wheel_joint: origin xyz=0.2 0 -0.15 rpy=0 0 0 -> xyz=0.2 0 -0.5 rpy=0 0 0
- joint base_joint: origin xyz=0 0 0.2 rpy=0 0 0 -> xyz=0 0 0.6 rpy=0 0 0
- joint base_left_wheel_joint: origin xyz=-0.1 0.2 -0.1 rpy=0 0 0 -> xyz=-0.0 0.2 -0.5 rpy=0 0 0
- joint base_right_wheel_joint: origin xyz=-0.1 -0.2 -0.1 rpy=0 0 0 -> xyz=-0.0 -0.2 -0.5 rpy=0 0 0
- joint base_scan_joint: origin xyz=0 0 0.13 rpy=0 0 0 -> xyz=0.5 0 -0.25 rpy=0 0 0

Commit message: fix

File: lucia_description/urdf/lucia.urdf (robot description, URDF)
Before this commit: robot lucia, 6 links, 5 joints
Links:
- removed link base_scan
- added link laser_front; visual cylinder length=0.06 radius=0.1
Joints:
- joint base_scan_joint: child base_scan -> laser_front

Commit message: add: laser_rear

File: lucia_description/urdf/lucia.urdf (robot description, URDF)
Before this commit: robot lucia, 6 links, 5 joints
Links:
- added link laser_rear; visual cylinder length=0.06 radius=0.1
Joints:
- removed joint base_scan_joint
- added joint laser_front_joint: type fixed, parent base_link, child laser_front, origin xyz=0.5 0 -0.25 rpy=0 0 0
- added joint laser_rear_joint: type fixed, parent base_link, child laser_rear, origin xyz=-0.5 0 -0.25 rpy=0 0 0

Commit message: fix

File: lucia_description/urdf/lucia.urdf (robot description, URDF)
Before this commit: robot lucia, 7 links, 6 joints
Joints:
- joint laser_rear_joint: origin xyz=-0.5 0 -0.25 rpy=0 0 0 -> xyz=-0.5 0 -0.25 rpy=0 0 3.14

Commit message: fix

File: lucia_description/urdf/lucia.urdf (robot description, URDF)
Before this commit: robot lucia, 7 links, 6 joints
Links:
- added link lsc_mount; visual cylinder length=0.06 radius=0.1
Joints:
- added joint lsc_mount_joint: type fixed, parent base_link, child lsc_mount, origin xyz=0.0 0 -0.25 rpy=0 0 0
- joint laser_front_joint: origin xyz=0.5 0 -0.25 rpy=0 0 0 -> xyz=0.5 0 0 rpy=0 0 0; parent base_link -> lsc_mount
- joint laser_rear_joint: origin xyz=-0.5 0 -0.25 rpy=0 0 3.14 -> xyz=-0.5 0 0 rpy=0 0 3.14; parent base_link -> lsc_mount
