Commit message: fix

File: urdf/lucia.urdf (robot description, URDF)
Before this commit: robot lucia, 8 links, 7 joints
Links:
- removed link caster_wheel
- link left_wheel: geometry visual cylinder length=0.1 radius=0.3
- link right_wheel: geometry visual cylinder length=0.1 radius=0.3
Joints:
- removed joint base_caster_wheel_joint
- joint base_left_wheel_joint: origin xyz=-0.0 0.2 -0.5 rpy=0 0 0 -> xyz=0.0 0.2 -0.5 rpy=0 0 0
- joint base_right_wheel_joint: origin xyz=-0.0 -0.2 -0.5 rpy=0 0 0 -> xyz=0.0 -0.2 -0.5 rpy=0 0 0

Commit message: fix

File: urdf/lucia.urdf (robot description, URDF)
Before this commit: robot lucia, 7 links, 6 joints
Links:
- link base_link: geometry visual cylinder length=1.1 radius=0.5
- link left_wheel: geometry visual cylinder length=0.1 radius=0.2
- link right_wheel: geometry visual cylinder length=0.1 radius=0.2
Joints:
- joint base_joint: origin xyz=0 0 0.6 rpy=0 0 0 -> xyz=0 0 0.55 rpy=0 0 0
- joint base_left_wheel_joint: origin xyz=0.0 0.2 -0.5 rpy=0 0 0 -> xyz=0.0 0.3 -0.5 rpy=0 0 0
- joint base_right_wheel_joint: origin xyz=0.0 -0.2 -0.5 rpy=0 0 0 -> xyz=0.0 -0.3 -0.5 rpy=0 0 0

Commit message: fix

File: urdf/lucia.urdf (robot description, URDF)
Before this commit: robot lucia, 7 links, 6 joints
Joints:
- joint base_joint: origin xyz=0 0 0.55 rpy=0 0 0 -> xyz=0.0 0.0 0.010 rpy=0 0 0

Commit message: fix

File: urdf/lucia.urdf (robot description, URDF)
Before this commit: robot lucia, 7 links, 6 joints
Joints:
- joint base_joint: origin xyz=0.0 0.0 0.010 rpy=0 0 0 -> xyz=0.0 0.0 0.5 rpy=0 0 0
- joint lsc_mount_joint: origin xyz=0.0 0 -0.25 rpy=0 0 0 -> xyz=0.0 0 0.25 rpy=0 0 0

Commit message: fix

File: urdf/lucia.urdf (robot description, URDF)
Before this commit: robot lucia, 7 links, 6 joints
Joints:
- joint lsc_mount_joint: origin xyz=0.0 0 0.25 rpy=0 0 0 -> xyz=0.0 0 -0.25 rpy=0 0 0

Commit message: fix

File: urdf/lucia.urdf (robot description, URDF)
Before this commit: robot lucia, 7 links, 6 joints
Joints:
- joint base_joint: origin xyz=0.0 0.0 0.5 rpy=0 0 0 -> xyz=0.0 0.0 0.55 rpy=0 0 0

Commit message: fix

File: urdf/lucia.urdf (robot description, URDF)
Before this commit: robot lucia, 7 links, 6 joints
Links:
- link left_wheel: geometry visual cylinder length=0.05 radius=0.1
- link right_wheel: geometry visual cylinder length=0.05 radius=0.1
Joints:
- joint base_joint: origin xyz=0.0 0.0 0.55 rpy=0 0 0 -> xyz=0.0 0.0 0.6 rpy=0 0 0

Commit message: fix

File: urdf/lucia.urdf (robot description, URDF)
Before this commit: robot lucia, 7 links, 6 joints
Links:
- added link camera_link; visual box size=0.05 0.1 0.03
Joints:
- added joint camera_joint: type fixed, parent base_link, child camera_link, origin xyz=0.4 0 0.3 rpy=0 0 0

Commit message: add: spina

File: urdf/lucia.urdf (robot description, URDF)
Before this commit: robot lucia, 8 links, 7 joints
Links:
- added link module1_lower_link, mass 0.1; collision cylinder length=0.02 radius=0.1; visual cylinder length=0.02 radius=0.1
- added link module1_pich_link, mass 0.05
- added link module1_roll_link, mass 0.05
- added link module1_upper_link, mass 0.1; collision cylinder length=0.02 radius=0.1; visual cylinder length=0.02 radius=0.1
- added link module2_lower_link, mass 0.1; collision cylinder length=0.02 radius=0.1; visual cylinder length=0.02 radius=0.1
- added link module2_pich_link, mass 0.05
- added link module2_roll_link, mass 0.05
- added link module2_upper_link, mass 0.1; collision cylinder length=0.02 radius=0.1; visual cylinder length=0.02 radius=0.1
- added link module3_lower_link, mass 0.1; collision cylinder length=0.02 radius=0.1; visual cylinder length=0.02 radius=0.1
- added link module3_pich_link, mass 0.05
- added link module3_roll_link, mass 0.05
- added link module3_upper_link, mass 0.1; collision cylinder length=0.02 radius=0.1; visual cylinder length=0.02 radius=0.1
- added link module4_lower_link, mass 0.1; collision cylinder length=0.02 radius=0.1; visual cylinder length=0.02 radius=0.1
- added link module4_pich_link, mass 0.05
- added link module4_roll_link, mass 0.05
- added link module4_upper_link, mass 0.1; collision cylinder length=0.02 radius=0.1; visual cylinder length=0.02 radius=0.1
- added link module5_lower_link, mass 0.1; collision cylinder length=0.02 radius=0.1; visual cylinder length=0.02 radius=0.1
- added link module5_pich_link, mass 0.05
- added link module5_roll_link, mass 0.05
- added link module5_upper_link, mass 0.1; collision cylinder length=0.02 radius=0.1; visual cylinder length=0.02 radius=0.1
- added link module6_lower_link, mass 0.1; collision cylinder length=0.02 radius=0.1; visual cylinder length=0.02 radius=0.1
- added link module6_pich_link, mass 0.05
- added link module6_roll_link, mass 0.05
- added link module6_upper_link, mass 0.1; collision cylinder length=0.02 radius=0.1; visual cylinder length=0.02 radius=0.1
Joints:
- added joint base_link_TO_module1_lower_link: type fixed, parent base_link, child module1_lower_link, origin xyz=0 0 0 rpy=0 0 0
- added joint base_link_TO_module2_lower_link: type fixed, parent module1_upper_link, child module2_lower_link, origin xyz=0 0 0 rpy=0 0 0
- added joint base_link_TO_module3_lower_link: type fixed, parent module2_upper_link, child module3_lower_link, origin xyz=0 0 0 rpy=0 0 0
- added joint base_link_TO_module4_lower_link: type fixed, parent module3_upper_link, child module4_lower_link, origin xyz=0 0 0 rpy=0 0 0
- added joint base_link_TO_module5_lower_link: type fixed, parent module4_upper_link, child module5_lower_link, origin xyz=0 0 0 rpy=0 0 0
- added joint base_link_TO_module6_lower_link: type fixed, parent module5_upper_link, child module6_lower_link, origin xyz=0 0 0 rpy=0 0 0
- added joint module1_gimbal_pitch: type revolute, parent module1_roll_link, child module1_pich_link, origin xyz=0 0 0 rpy=0 0 0, axis 0 1 0, limit lower=-0.5236 upper=0.5236 effort=1 velocity=1
- added joint module1_gimbal_roll: type revolute, parent module1_lower_link, child module1_roll_link, origin xyz=0 0 0.075 rpy=0 0 0, axis 1 0 0, limit lower=-0.5236 upper=0.5236 effort=1 velocity=1
- added joint module1_pich_link_TO_module1_upper_link: type fixed, parent module1_pich_link, child module1_upper_link, origin xyz=0 0 0.075 rpy=0 0 0
- added joint module2_gimbal_pitch: type revolute, parent module2_roll_link, child module2_pich_link, origin xyz=0 0 0 rpy=0 0 0, axis 0 1 0, limit lower=-0.5236 upper=0.5236 effort=1 velocity=1
- added joint module2_gimbal_roll: type revolute, parent module2_lower_link, child module2_roll_link, origin xyz=0 0 0.075 rpy=0 0 0, axis 1 0 0, limit lower=-0.5236 upper=0.5236 effort=1 velocity=1
- added joint module2_pich_link_TO_module2_upper_link: type fixed, parent module2_pich_link, child module2_upper_link, origin xyz=0 0 0.075 rpy=0 0 0
- added joint module3_gimbal_pitch: type revolute, parent module3_roll_link, child module3_pich_link, origin xyz=0 0 0 rpy=0 0 0, axis 0 1 0, limit lower=-0.5236 upper=0.5236 effort=1 velocity=1
- added joint module3_gimbal_roll: type revolute, parent module3_lower_link, child module3_roll_link, origin xyz=0 0 0.075 rpy=0 0 0, axis 1 0 0, limit lower=-0.5236 upper=0.5236 effort=1 velocity=1
- added joint module3_pich_link_TO_module3_upper_link: type fixed, parent module3_pich_link, child module3_upper_link, origin xyz=0 0 0.075 rpy=0 0 0
- added joint module4_gimbal_pitch: type revolute, parent module4_roll_link, child module4_pich_link, origin xyz=0 0 0 rpy=0 0 0, axis 0 1 0, limit lower=-0.5236 upper=0.5236 effort=1 velocity=1
- added joint module4_gimbal_roll: type revolute, parent module4_lower_link, child module4_roll_link, origin xyz=0 0 0.075 rpy=0 0 0, axis 1 0 0, limit lower=-0.5236 upper=0.5236 effort=1 velocity=1
- added joint module4_pich_link_TO_module4_upper_link: type fixed, parent module4_pich_link, child module4_upper_link, origin xyz=0 0 0.075 rpy=0 0 0
- added joint module5_gimbal_pitch: type revolute, parent module5_roll_link, child module5_pich_link, origin xyz=0 0 0 rpy=0 0 0, axis 0 1 0, limit lower=-0.5236 upper=0.5236 effort=1 velocity=1
- added joint module5_gimbal_roll: type revolute, parent module5_lower_link, child module5_roll_link, origin xyz=0 0 0.075 rpy=0 0 0, axis 1 0 0, limit lower=-0.5236 upper=0.5236 effort=1 velocity=1
- added joint module5_pich_link_TO_module5_upper_link: type fixed, parent module5_pich_link, child module5_upper_link, origin xyz=0 0 0.075 rpy=0 0 0
- added joint module6_gimbal_pitch: type revolute, parent module6_roll_link, child module6_pich_link, origin xyz=0 0 0 rpy=0 0 0, axis 0 1 0, limit lower=-0.5236 upper=0.5236 effort=1 velocity=1
- added joint module6_gimbal_roll: type revolute, parent module6_lower_link, child module6_roll_link, origin xyz=0 0 0.075 rpy=0 0 0, axis 1 0 0, limit lower=-0.5236 upper=0.5236 effort=1 velocity=1
- added joint module6_pich_link_TO_module6_upper_link: type fixed, parent module6_pich_link, child module6_upper_link, origin xyz=0 0 0.075 rpy=0 0 0

Commit message: fix

File: urdf/lucia.urdf (robot description, URDF)
Before this commit: robot lucia, 32 links, 31 joints
Joints:
- joint base_link_TO_module1_lower_link: origin xyz=0 0 0 rpy=0 0 0 -> xyz=0 0 0.6 rpy=0 0 0

Commit message: fix

File: urdf/lucia.urdf (robot description, URDF)
Before this commit: robot lucia, 32 links, 31 joints
Links:
- added link vital_arm_link; visual cylinder length=0.1 radius=0.05
Joints:
- added joint vital_arm_joint: type fixed, parent module6_upper_link, child vital_arm_link, origin xyz=0 0 0 rpy=0 0 0

Commit message: fix

File: urdf/lucia.urdf (robot description, URDF)
Before this commit: robot lucia, 33 links, 32 joints
Links:
- link vital_arm_link: geometry visual cylinder length=0.15 radius=0.05
Joints:
- joint vital_arm_joint: origin xyz=0 0 0 rpy=0 0 0 -> xyz=0 0 0.05 rpy=0 0 0

Commit message: add: camera

File: urdf/lucia.urdf (robot description, URDF)
Before this commit: robot lucia, 33 links, 32 joints
Joints:
- joint camera_joint: parent base_link -> module6_upper_link

Commit message: fix

File: urdf/lucia.urdf (robot description, URDF)
Before this commit: robot lucia, 33 links, 32 joints
Joints:
- joint camera_joint: origin xyz=0.4 0 0.3 rpy=0 0 0 -> xyz=0.05 0 0.05 rpy=0 0 0

Commit message: fix

File: urdf/lucia.urdf (robot description, URDF)
Before this commit: robot lucia, 33 links, 32 joints
Joints:
- joint camera_joint: origin xyz=0.05 0 0.05 rpy=0 0 0 -> xyz=0.4 0 0.3 rpy=0 0 0; parent module6_upper_link -> base_link
